Commit message: gripper move

File: src/tm_description/urdf/tm.transmission.xacro (robot description, xacro)
@@ -56,13 +56,13 @@
       </actuator>
     </transmission>
-    <transmission name="${prefix}gripper_trans">
-      <type>transmission_interface/SimpleTransmission</type>
-      <joint name="${prefix}gripper_joint">
-        <hardwareInterface>PositionJointInterface</hardwareInterface>
-      </joint>
-      <actuator name="${prefix}gripper_motor">
-        <mechanicalReduction>1</mechanicalReduction>
-      </actuator>
-    </transmission>
+<!--    <transmission name="${prefix}gripper_trans">-->
+<!--      <type>transmission_interface/SimpleTransmission</type>-->
+<!--      <joint name="${prefix}gripper_joint">-->
+<!--        <hardwareInterface>PositionJointInterface</hardwareInterface>-->
+<!--      </joint>-->
+<!--      <actuator name="${prefix}gripper_motor">-->
+<!--        <mechanicalReduction>1</mechanicalReduction>-->
+<!--      </actuator>-->
+<!--    </transmission>-->
     <transmission name="${prefix}finger_r_trans">
       <type>transmission_interface/SimpleTransmission</type>

File: src/tm_description/urdf/tm700.urdf.xacro (robot description, xacro)
@@ -275,5 +275,5 @@
     <property name="gripper_joint_x" value="0" />
     <property name="gripper_joint_y" value="0" />
-    <property name="gripper_joint_z" value="0.055" />
+    <property name="gripper_joint_z" value="0.058" />
     <property name="gripper_roll" value="0" />
     <property name="gripper_pitch" value="${-pi/2}" />
@@ -281,5 +281,5 @@
     <property name="finger_bias_x" value="-0.07285" />
     <property name="finger_bias_y" value="0.005" />
-    <property name="finger_bias_z" value="0.07" />
+    <property name="finger_bias_z" value="0.068" />
     <property name="finger_r_joint_x" value="${finger_bias_x+0.07285}" />
     <property name="finger_r_joint_y" value="${finger_bias_y+0}" />
@@ -310,5 +310,5 @@
         </collision>
     </link>
-    <joint name="${prefix}gripper_joint" type="revolute">
+    <joint name="${prefix}gripper_joint" type="fixed">
         <origin rpy="0 0 0" xyz="${gripper_joint_x} ${gripper_joint_y} ${gripper_joint_z}"/>
         <parent link="${prefix}wrist_3_link"/>
@@ -339,9 +339,10 @@
         </collision>
     </link>
+<!--prismatic-->
     <joint name="${prefix}finger_r_joint" type="prismatic">
         <origin rpy="0 0 0" xyz="${finger_r_joint_x} ${finger_r_joint_y} ${finger_r_joint_z}"/>
         <parent link="${prefix}gripper_link"/>
         <child link="${prefix}finger_r_link"/>
-        <axis xyz="0 1 0"/>
+        <axis xyz="1 0 0"/>
         <limit effort="1" lower="-1" upper="0" velocity="1"/>
     </joint>
@@ -368,9 +369,10 @@
         </collision>
     </link>
+<!--prismatic-->
     <joint name="${prefix}finger_l_joint" type="prismatic">
         <origin rpy="0 0 0" xyz="${finger_l_joint_x} ${finger_l_joint_y} ${finger_l_joint_z}"/>
         <parent link="${prefix}gripper_link"/>
         <child link="${prefix}finger_l_link"/>
-        <axis xyz="0 1 0"/>
+        <axis xyz="1 0 0"/>
         <limit effort="1" lower="0" upper="1" velocity="1"/>
     </joint>
